File: hardware/board_2a/conf.kicad_sch (KiCad schematic)
At the start: 58 parts, among them J7 Conn_02x04_Odd_Even, Q1 Q_NPN_BEC, SW1 204-124ST, SW2 SW_Push, SW4 SW_Push, SW6 SW_Push, U1 Ti60F256, U14 Si5351A-B-GT, U15 MC2520Z 25MHz, U4 W25Q128JWS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

Commit message: Update hardware/board_2a
Connections:
- net GND: now also J7.3 (Pin_3)
- net SD_VDD_SEL_3V3 renamed SD_VCCIO_SEL_3V3
- no-connect marks 51 -> 50
Changed lines of the file:
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@@
+	)
+	(junction
+		(at 128.27 64.135)
+		(diameter 0)
+		(color 0 0 0 0)
 	)
 	(junction
@@
 	)
 	(no_connect
-		(at 130.81 66.675)
-	)
-	(no_connect
 		(at 203.2 82.55)
 	)
@@
 	(wire
 		(pts
+			(xy 130.81 66.675) (xy 128.27 66.675)
+		)
+		(stroke
+			(width 0)
+			(type default)
+		)
+	)
+	(wire
+		(pts
 			(xy 232.41 140.335) (xy 245.11 140.335)
 		)
@@
 	(wire
 		(pts
+			(xy 128.27 64.135) (xy 120.65 64.135)
+		)
+		(stroke
+			(width 0)
+			(type default)
+		)
+	)
+	(wire
+		(pts
 			(xy 37.465 178.435) (xy 37.465 181.61)
 		)
@@
 	(wire
 		(pts
-			(xy 130.81 64.135) (xy 120.65 64.135)
+			(xy 130.81 64.135) (xy 128.27 64.135)
 		)
 		(stroke
@@
 		(pts
 			(xy 168.91 40.005) (xy 168.91 41.275)
+		)
+		(stroke
+			(width 0)
+			(type default)
+		)
+	)
+	(wire
+		(pts
+			(xy 128.27 66.675) (xy 128.27 64.135)
 		)
 		(stroke
@@
 		)
 	)
-	(global_label "SD_VDD_SEL_3V3"
+	(global_label "SD_VCCIO_SEL_3V3"
 		(shape input)
 		(at 203.2 99.695 0)
