File: hardware/board_2a/endeavour2.kicad_pcb (KiCad board)
At the start: 6 copper layers, 100 x 85 mm, 230 parts, among them J1 HDMI_A, J10 jumper_power_source, J11 Conn_GPIO, J12 jumper_5v, J13 Conn_power, J2 USB_C_Receptacle_USB2.0, J3 SJ-3523-SMT, J4 USB_A, J5 USB_A, J6 Micro_SD_Card_Det2, J7 Conn_02x04_Odd_Even, J8 Conn_01x02, J9 USB_C_Receptacle_USB2.0, Q1 Q_NPN_BEC, SW1 204-124ST, SW2 SW_Push, SW4 SW_Push, SW6 SW_Push, SW7 SW_SPDT, SW9 SW_SPDT, U1 Ti60F256, U10 MCP4728, U11 LM4811, U12 PCF85063AT/AY, U13 STUSB4500QTR, U14 Si5351A-B-GT, U15 MC2520Z 25MHz, U16 SN74LVC1T45DCK, U17 TPS2116DRLR, U18 TPS562211DRLR, U19 TPS562211DRLR, U2 IM8G16D3FFBG, U20 TPS562211DRLR, U21 TPS562211DRLR, U22 TPS562211DRLR, U3 TFP410PAP, U4 W25Q128JWS, U5 FT2232HL, U6 AP22653W6-7, U7 AP22653W6-7, U8 ESP32-C3-WROOM-02-N4, U9 AP22653W6-7, Y1 12MHz, Y2 Crystal, Y3 25MHz

Commit message: PCB update
Parts:
- moved C14 0.08 mm to (161.9, 113.8)
Routing:
- net +1V35: track 94.1 -> 94.9 mm, vias 39 -> 38
- net Net-(JP1-C): track 23.6 -> 22.8 mm
- net GPIO_A9: track 26.4 -> 25.8 mm
- net GND: vias 209 -> 203
- net DDR_DQ2: vias 3 -> 2
- added copper zone on F.Cu, net (none)
Other:
- board text added: "SND PWR"
- board text added: "STATUS"
- board text removed: "NSTATUS"

Commit message: Update hardware/board_2a
Parts:
- added D10: D_TVS, Diode_SMD:D_0603_1608Metric, B.Cu at (137.9, 126.0)
- added D11: D_TVS, Diode_SMD:D_0603_1608Metric, B.Cu at (137.9, 124.2)
- added D12: D_TVS, Diode_SMD:D_0603_1608Metric, B.Cu at (184.1, 119.1)
- added D13: D_TVS, Diode_SMD:D_0603_1608Metric, B.Cu at (184.0, 122.6)
- added D14: D_TVS, Diode_SMD:D_0603_1608Metric, B.Cu at (174.6, 136.1)
- added D15: D_TVS, Diode_SMD:D_0603_1608Metric, B.Cu at (171.0, 136.1)
Routing:
- net GND: track 441.7 -> 455.6 mm, vias 203 -> 204
- net USBC_D+: track 35.0 -> 36.0 mm
- net USB1_D-: track 42.0 -> 42.9 mm
- net USBC_D-: track 35.7 -> 36.5 mm
- net USB1_D+: track 43.5 -> 44.3 mm
- net USB2_D+: track 49.5 -> 50.2 mm
- net USB2_D-: track 48.9 -> 49.7 mm

Commit message: Update hardware/board_2a
Parts:
- added C4: 1uF, Capacitor_SMD:C_0603_1608Metric, B.Cu at (142.6, 94.7)
- added C60: 0.1uF, Capacitor_SMD:C_0603_1608Metric, B.Cu at (141.6, 101.3)
- added J14: Conn_01x04_Pin, Connector_PinHeader_2.54mm:PinHeader_1x04_P2.54mm_Vertical, F.Cu at (191.9, 73.5)
- added U23: SN74LVC1T45DCK, Package_TO_SOT_SMD:SOT-363_SC-70-6, B.Cu at (163.8, 142.8)
- added U24: SN74LVC1T45DCK, Package_TO_SOT_SMD:SOT-363_SC-70-6, B.Cu at (181.2, 76.9)
- added U25: SN74LVC1T45DCK, Package_TO_SOT_SMD:SOT-363_SC-70-6, B.Cu at (174.3, 71.5)
- C19: value 10uF -> 0.1uF
- C23, C8: value 0.1uF -> 4.7uF
- C9: value 4.7uF -> 1uF
- D7, D8: footprint Diode_SMD:D_0603_1608Metric -> Diode_SMD:D_SOD-323
- L1, L2, L3, L4, L5: footprint Inductor_SMD:L_0603_1608Metric -> Inductor_SMD:L_1008_2520Metric
- R58, R59: value 75 -> 10K
- R64: value 11.7K -> 23.2K
- R65: value 20K -> 40.2K
- R66: value 25K -> 24.9K
- R68: value 40K -> 40.2K
- R70: value 73.3K -> 73.2K
- R72: value 45K -> 45.3K
- moved R58 13.6 mm to (181.2, 74.0)
- moved C9 12.6 mm to (153.1, 102.8)
- moved R59 11.6 mm to (169.8, 80.3), turned to 180 degrees
- moved R57 10.1 mm to (172.8, 77.3), turned to -90 degrees
- moved C12 7.36 mm to (148.2, 98.0), turned to 90 degrees
- moved C10 5.91 mm to (152.2, 94.8), turned to 90 degrees
- moved C7 5.91 mm to (147.4, 101.2), turned to -90 degrees
- moved R60 5.82 mm to (169.8, 74.2), turned to 180 degrees
- moved C11 3.63 mm to (141.0, 94.7), turned to -90 degrees
- moved C80 2.69 mm to (116.6, 109.1)
- moved C85 2.67 mm to (114.6, 109.1)
- moved L4 1.25 mm to (119.1, 110.8), turned to 90 degrees
- moved C6 1.11 mm to (141.6, 102.8)
- moved C77 1.07 mm to (135.9, 90.3)
- moved C82 1.07 mm to (138.0, 90.3)
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Connections:
- net SD_VDD_SEL_3V3 renamed SD_VCCIO_SEL_3V3
- C22 pad 1: SD_VDD -> SD_VCCIO
- C66 pad 1: SD_VDD -> +3V3
- J6 pad 4: SD_VDD -> +3V3
- J7 pad 3: unconnected-(J7-Pin_3-Pad3) -> GND
- R55 pad 1: Net-(U1H-GPIOR_15) -> ESP32_TX
- R56 pad 1: Net-(U1H-GPIOR_17) -> ESP32_RX_3V3
- R57 pad 1: Net-(U1H-GPIOR_16) -> ESP32_SPI_BOOT_3V3
- R57 pad 2: Net-(U8-IO10) -> Net-(U8-IO9)
- R58 pad 1: Net-(U1H-GPIOR_19) -> +3V3
- R59 pad 1: Net-(U1H-GPIOR_14) -> +3V3
- R59 pad 2: Net-(U8-IO3) -> Net-(U8-IO8)
- R60 pad 1: Net-(U1H-GPIOR_20) -> ESP32_IO4
- R61 pad 1: Net-(U1H-GPIOR_18) -> ESP32_IO7
- R62 pad 1: Net-(U1H-GPIOR_13) -> ESP32_IO6
- R63 pad 1: Net-(U1H-GPIOR_12) -> ESP32_IO5
- U1 pad A11: unconnected-(U1G-GPIOT_P_13-PadA11) -> ESP32_SPI_BOOT
- U1 pad A12: Net-(U1H-GPIOR_12) -> 3V3_SDA
- U1 pad A13: Net-(U1H-GPIOR_13) -> 3V3_SCL
- U1 pad A14: Net-(U1H-GPIOR_15) -> ESP32_IO5
- U1 pad A15: Net-(U1H-GPIOR_16) -> ESP32_IO7
- U1 pad B10: unconnected-(U1G-GPIOT_P_10_CLK7_P-PadB10) -> ESP32_EN
- U1 pad B12: unconnected-(U1G-GPIOT_P_16_EXTFB-PadB12) -> ESP32_RX
- U1 pad B14: Net-(U1H-GPIOR_17) -> ESP32_IO6
- U1 pad B3: SD_VDD -> SD_VCCIO
- U1 pad C13: Net-(U1H-GPIOR_14) -> ESP32_IO4
- U1 pad C14: Net-(U1H-GPIOR_19) -> unconnected-(U1H-GPIOR_19-PadC14)
- U1 pad D13: Net-(U1H-GPIOR_18) -> ESP32_TX
- U1 pad E13: Net-(U1H-GPIOR_20) -> unconnected-(U1H-GPIOR_20-PadE13)
- U1 pad E14: ESP32_EN -> SND_SHDN
- U1 pad M12: 3V3_SDA -> unconnected-(U1K-GPIOR_23-PadM12)
- U1 pad N12: 3V3_SCL -> unconnected-(U1K-GPIOR_26-PadN12)
- U1 pad R16: SND_SHDN -> unconnected-(U1K-GPIOR_21-PadR16)
- U11 pad 7: SND_SHDN -> Net-(U11-SHDN)
- U16 pad 6: +1V35 -> +1V8
- U17 pad 2: SD_VDD -> SD_VCCIO
- U17 pad 7: SD_VDD -> SD_VCCIO
- U8 pad 10: Net-(U8-IO10) -> unconnected-(U8-IO10-Pad10)
- U8 pad 15: Net-(U8-IO3) -> unconnected-(U8-IO3-Pad15)
- U8 pad 7: unconnected-(U8-IO8-Pad7) -> Net-(U8-IO8)
- U8 pad 8: unconnected-(U8-IO9-Pad8) -> Net-(U8-IO9)
Routing:
- net +1V35: track 94.9 -> 144.5 mm
- net ESP32_SPI_BOOT: track 0.00 -> 39.4 mm, vias 0 -> 2
- net ESP32_RX: track 0.00 -> 37.5 mm, vias 0 -> 2
- net SD_VDD: track 37.1 -> 0.00 mm, vias 3 -> 0
- net Net-(U1H-GPIOR_14): track 34.9 -> 0.00 mm, vias 1 -> 0
- net ESP32_TX: track 0.00 -> 33.6 mm, vias 0 -> 2
- net Net-(U1H-GPIOR_15): track 32.0 -> 0.00 mm, vias 1 -> 0
- net Net-(U1H-GPIOR_17): track 31.7 -> 0.00 mm, vias 1 -> 0
- net ESP32_IO4: track 0.00 -> 31.6 mm, vias 0 -> 1
- net Net-(U1H-GPIOR_16): track 29.6 -> 0.00 mm, vias 1 -> 0
- net GND: track 455.6 -> 483.6 mm, vias 204 -> 207
- net ESP32_IO5: track 0.00 -> 27.9 mm, vias 0 -> 1
- net ESP32_IO6: track 0.00 -> 27.2 mm, vias 0 -> 1
- net Net-(U1H-GPIOR_12): track 25.8 -> 0.00 mm, vias 2 -> 0
- net ESP32_IO7: track 0.00 -> 24.7 mm, vias 0 -> 1
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- removed copper zone on F.Cu, net Net-(J12-Pin_3)
Other:
- board text added: "CERR"
- board text added: "I2C"
- board text added: "SCL"
- board text added: "SDA"
- board text removed: "STATUS"
