File: hardware/board_2a/endeavour2.kicad_sch (KiCad schematic)
At the start: 19 parts, among them J10 jumper_power_source, J11 Conn_GPIO, J2 USB_C_Receptacle_USB2.0, J9 USB_C_Receptacle_USB2.0, SW9 SW_SPDT, U1 Ti60F256, U13 STUSB4500QTR

Commit message: Update hardware/board_2a
Parts:
- added D10, D11: D_TVS, Diode_SMD:D_0603_1608Metric, symbol Device:D_TVS
Connections:
- net GND: now also D10.1 (A1), D11.1 (A1)
- net USBC_D+: now also D11.2 (A2)
- net USBC_D-: now also D10.2 (A2)

Commit message: Update hardware/board_2a
Parts:
- added J14: Conn_01x04_Pin, Connector_PinHeader_2.54mm:PinHeader_1x04_P2.54mm_Vertical, symbol Connector:Conn_01x04_Pin
- added U16, U24, U25: SN74LVC1T45DCK, Package_TO_SOT_SMD:SOT-363_SC-70-6, symbol Logic_LevelTranslator:SN74LVC1T45DCK
Connections:
- net +1V8: now also U16.6 (VCCB), U24.6 (VCCB), U25.6 (VCCB)
- net +3V3: now also J14.4 (Pin_4), U16.1 (VCCA), U24.1 (VCCA), U25.1 (VCCA)
- net 3V3_SCL: now also J14.2 (Pin_2)
- net 3V3_SDA: now also J14.3 (Pin_3)
- net GND: now also J14.1 (Pin_1), U16.2 (GND), U16.5 (DIR), U24.2 (GND), U24.5 (DIR), U25.2 (GND), U25.5 (DIR)
- net ESP32_SPI_BOOT: now reaches U1.A11 (GPIOT_P_13)
- net ESP32_SPI_BOOT: now also U25.4 (B)
- net ESP32_EN: now reaches U1.B10 (GPIOT_P_10_CLK7_P)
- net ESP32_EN: now also U16.4 (B)
- net ESP32_RX: now reaches U1.B12 (GPIOT_P_16_EXTFB)
- net ESP32_RX: now also U24.4 (B)
- new net ESP32_EN_3V3: U16.3 (A)
- new net ESP32_RX_3V3: U24.3 (A)
- new net ESP32_SPI_BOOT_3V3: U25.3 (A)
- no-connect marks 32 -> 29
Other:
- moved on the sheet: J11, R2, U1F, U1G
