File: hardware/board_2a/peripherals.kicad_sch (KiCad schematic)
At the start: 54 parts, among them J3 SJ-3523-SMT, J4 USB_A, J5 USB_A, J6 Micro_SD_Card_Det2, J8 Conn_01x02, SW7 SW_SPDT, U1 Ti60F256, U10 MCP4728, U11 LM4811, U12 PCF85063AT/AY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

Commit message: Update hardware/board_2a
Parts:
- added D12, D13, D14, D15: D_TVS, Diode_SMD:D_0603_1608Metric, symbol Device:D_TVS
Connections:
- net GND: now also D12.1 (A1), D13.1 (A1), D14.1 (A1), D15.1 (A1)
- net USB1_D+: now also D12.2 (A2)
- net USB1_D-: now also D13.2 (A2)
- net USB2_D+: now also D14.2 (A2)
- net USB2_D-: now also D15.2 (A2)

Commit message: Update hardware/board_2a
Parts:
- removed U16: SN74LVC1T45DCK, Package_TO_SOT_SMD:SOT-363_SC-70-6, symbol Logic_LevelTranslator:SN74LVC1T45DCK
- added C4: 1uF, Capacitor_SMD:C_0603_1608Metric, symbol Device:C
- added U23: SN74LVC1T45DCK, Package_TO_SOT_SMD:SOT-363_SC-70-6, symbol Logic_LevelTranslator:SN74LVC1T45DCK
- D7, D8: footprint Diode_SMD:D_0603_1608Metric -> Diode_SMD:D_SOD-323
- R58, R59: value 75 -> 10K
Connections:
- net +1V35: now also U23.6 (VCCB)
- net +3V3: now also C66.1, J6.4 (VDD), R58.1, R59.1, C4.1
- net 3V3_SCL: now also U1.A13 (GPIOR_13); no longer U1.N12 (GPIOR_26)
- net 3V3_SDA: now also U1.A12 (GPIOR_12); no longer U1.M12 (GPIOR_23)
- net GND: now also C4.2, U23.2 (GND), U23.5 (DIR)
- net SND_SHDN: now also U23.4 (B); no longer U1.R16 (GPIOR_21), U11.7 (SHDN)
- net ESP32_IO5: now reaches U1.A14 (GPIOR_15)
- net ESP32_IO5: now also R63.1; no longer R55.1
- net ESP32_IO7: now reaches U1.A15 (GPIOR_16)
- net ESP32_IO7: now also R61.1; no longer R57.1
- net at R57.2: now also U8.8 (IO9); no longer U8.10 (IO10)
- net at C49.2, JP1.2 (C), U10.1 (VDD)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: now also U23.1 (VCCA)
- net ESP32_IO6: now reaches U1.B14 (GPIOR_17)
- net ESP32_IO6: now also R62.1; no longer R56.1
- net ESP32_TX: now reaches U1.D13 (GPIOR_18)
- net ESP32_TX: now also R55.1; no longer R61.1
- net at U8.15 (IO3): no longer R59.2
- net at U8.7 (IO8): now also R59.2
- net ESP32_IO4: now reaches U1.C13 (GPIOR_14)
- net ESP32_IO4: now also R60.1; no longer R59.1
- net at U1.E13 (GPIOR_20): no longer R60.1
- net at U1.C14 (GPIOR_19): no longer R58.1
- net SD_VDD renamed SD_VCCIO
- net SD_VCCIO: no longer C66.1, J6.4 (VDD)
- net SD_VDD_SEL_3V3 renamed SD_VCCIO_SEL_3V3
- new net: U11.7 (SHDN), U23.3 (A)
- new net ESP32_RX_3V3: R56.1
- new net ESP32_SPI_BOOT_3V3: R57.1
- no-connect marks 16 -> 21
Other:
- moved on the sheet: C47, C48, C49, C50, C51, C52, C66, J3, J8, JP1, R46, R47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
