File: hardware/board_2a/power.kicad_sch (KiCad schematic)
At the start: 63 parts, among them J12 jumper_5v, J13 Conn_power, U1 Ti60F256, U18 TPS562211DRLR, U19 TPS562211DRLR, U20 TPS562211DRLR, U21 TPS562211DRLR, U22 TPS562211DRLR

Commit message: Update hardware/board_2a
Parts:
- added C60: 0.1uF, Capacitor_SMD:C_0603_1608Metric, symbol Device:C
- C19: value 10uF -> 0.1uF
- C23, C8: value 0.1uF -> 4.7uF
- C9: value 4.7uF -> 1uF
- L1, L2, L3, L4, L5: footprint Inductor_SMD:L_0603_1608Metric -> Inductor_SMD:L_1008_2520Metric
- R64: value 11.7K -> 23.2K
- R65: value 20K -> 40.2K
- R66: value 25K -> 24.9K
- R68: value 40K -> 40.2K
- R70: value 73.3K -> 73.2K
- R72: value 45K -> 45.3K
Connections:
- net +0V95: now also C60.1
- net GND: now also C60.2
- net SD_VDD renamed SD_VCCIO
Changed lines of the file:
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@@
 	)
 	(junction
+		(at 132.715 27.305)
+		(diameter 0)
+		(color 0 0 0 0)
+	)
+	(junction
 		(at 35.56 59.055)
 		(diameter 0)
@@
 	)
 	(junction
+		(at 132.715 34.925)
+		(diameter 0)
+		(color 0 0 0 0)
+	)
+	(junction
 		(at 35.56 74.295)
 		(diameter 0)
@@
 	(wire
 		(pts
+			(xy 132.715 34.925) (xy 139.7 34.925)
+		)
+		(stroke
+			(width 0)
+			(type default)
+		)
+	)
+	(wire
+		(pts
 			(xy 94.615 85.09) (xy 94.615 89.535)
 		)
@@
 	(wire
 		(pts
+			(xy 132.715 27.305) (xy 139.7 27.305)
+		)
+		(stroke
+			(width 0)
+			(type default)
+		)
+	)
+	(wire
+		(pts
 			(xy 87.63 133.35) (xy 107.315 133.35)
 		)
@@
 		)
 	)
-	(global_label "SD_VDD"
+	(global_label "SD_VCCIO"
 		(shape input)
 		(at 35.56 99.06 180)
@@
 			)
 		)
-		(property "Value" "4.7uF"
+		(property "Value" "1uF"
 			(at 133.35 33.655 0)
 			(effects
@@
 			)
 		)
-		(property "Footprint" "Inductor_SMD:L_0603_1608Metric"
+		(property "Footprint" "Inductor_SMD:L_1008_2520Metric"
 			(at 238.76 81.28 0)
 			(effects
@@
 			)
 		)
-		(property "Value" "20K"
-			(at 240.03 137.795 0)
+		(property "Value" "40.2K"
+			(at 238.76 137.795 0)
 			(effects
 				(font
@@
 	(symbol
 		(lib_id "Device:C")
+		(at 139.7 31.115 0)
+		(unit 1)
+		(exclude_from_sim no)
+		(in_bom yes)
+		(on_board yes)
+		(dnp no)
+		(property "Reference" "C60"
+			(at 140.97 28.575 0)
+			(effects
+				(font
+					(size 1.27 1.27)
+				)
+				(justify left)
+			)
+		)
+		(property "Value" "0.1uF"
+			(at 140.335 33.655 0)
+			(effects
+				(font
+					(size 1.27 1.27)
+				)
+				(justify left)
+			)
+		)
+		(property "Footprint" "Capacitor_SMD:C_0603_1608Metric"
+			(at 140.6652 34.925 0)
+			(effects
+				(font
+					(size 1.27 1.27)
+				)
+				(hide yes)
+			)
+		)
+		(property "Datasheet" "~"
+			(at 139.7 31.115 0)
+			(effects
+				(font
+					(size 1.27 1.27)
+				)
+				(hide yes)
+			)
+		)
+		(property "Description" "Unpolarized capacitor"
+			(at 139.7 31.115 0)
+			(effects
+				(font
+					(size 1.27 1.27)
+				)
+				(hide yes)
+			)
+		)
+		(pin "1"
+		)
+		(pin "2"
+		)
+		(instances
+			(project "endeavour2"
+				(path "/3f72371b-702d-4dab-a6c7-f93a430e8a08/04a0083b-c019-4ec4-9f0e-50dd3ee28f0c"
+					(reference "C60")
+					(unit 1)
+				)
+			)
+		)
+	)
+	(symbol
+		(lib_id "Device:C")
 		(at 38.1 129.54 0)
 		(unit 1)
@@
 			)
 		)
-		(property "Value" "73.3K"
+		(property "Value" "73.2K"
 			(at 102.87 128.27 0)
 			(effects
@@
 			)
 		)
-		(property "Footprint" "Inductor_SMD:L_0603_1608Metric"
+		(property "Footprint" "Inductor_SMD:L_1008_2520Metric"
 			(at 238.125 123.825 0)
 			(effects
@@
 			)
 		)
-		(property "Footprint" "Inductor_SMD:L_0603_1608Metric"
+		(property "Footprint" "Inductor_SMD:L_1008_2520Metric"
 			(at 102.235 123.19 0)
 			(effects
@@
 			)
 		)
-		(property "Value" "40K"
-			(at 241.3 41.91 0)
+		(property "Value" "40.2K"
+			(at 240.03 42.545 0)
 			(effects
 				(font
@@
 			)
 		)
-		(property "Value" "11.7K"
+		(property "Value" "23.2K"
 			(at 238.76 128.905 0)
 			(effects
@@
 			)
 		)
-		(property "Value" "45K"
-			(at 104.14 171.45 0)
+		(property "Value" "45.3K"
+			(at 102.87 172.085 0)
 			(effects
 				(font
@@
 			)
 		)
-		(property "Footprint" "Inductor_SMD:L_0603_1608Metric"
+		(property "Footprint" "Inductor_SMD:L_1008_2520Metric"
 			(at 239.395 36.83 0)
 			(effects
@@
 			)
 		)
-		(property "Value" "0.1uF"
+		(property "Value" "4.7uF"
 			(at 97.79 26.67 0)
 			(effects
@@
 			)
 		)
-		(property "Value" "25K"
-			(at 240.665 86.36 0)
+		(property "Value" "24.9K"
+			(at 239.395 86.995 0)
 			(effects
 				(font
@@
 			)
 		)
-		(property "Footprint" "Inductor_SMD:L_0603_1608Metric"
+		(property "Footprint" "Inductor_SMD:L_1008_2520Metric"
 			(at 102.235 166.37 0)
 			(effects
@@
 			)
 		)
-		(property "Value" "0.1uF"
+		(property "Value" "4.7uF"
 			(at 125.095 26.035 0)
 			(effects
@@
 			)
 		)
-		(property "Value" "10uF"
+		(property "Value" "0.1uF"
 			(at 75.565 34.29 0)
 			(effects
