File: hardware/board_2a/ram.kicad_sch (KiCad schematic)
At the start: 36 parts, among them J1 HDMI_A, U1 Ti60F256, U2 IM8G16D3FFBG, U3 TFP410PAP, U9 AP22653W6-7

Commit message: Update hardware/board_2a
Connections:
- net ESP32_EN renamed SND_SHDN
Changed lines of the file:
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@@
+		)
+	)
+	(global_label "SND_SHDN"
+		(shape input)
+		(at 139.7 55.88 0)
+		(fields_autoplaced yes)
+		(effects
+			(font
+				(size 0.762 0.762)
+			)
+			(justify left)
+		)
+		(property "Intersheetrefs" "${INTERSHEET_REFS}"
+			(at 147.4423 55.88 0)
+			(effects
+				(font
+					(size 1.27 1.27)
+				)
+				(justify left)
+				(hide yes)
+			)
 		)
 	)
@@
 				(hide yes)
 			)
-		)
-	)
-	(global_label "ESP32_EN"
-		(shape input)
-		(at 139.7 55.88 0)
-		(fields_autoplaced yes)
-		(effects
-			(font
-				(size 0.762 0.762)
-			)
-			(justify left)
-		)
-		(property "Intersheetrefs" "${INTERSHEET_REFS}"
-			(at 147.1882 55.88 0)
-			(effects
-				(font
-					(size 1.27 1.27)
-				)
-				(justify left)
-				(hide yes)
-			)
