File: hardware/board_2a/endeavour2_upd.kicad_pcb (KiCad board)
At the start: 6 copper layers, 100 x 85 mm, 242 parts, among them J1 HDMI_A, J10 jumper_power_source, J11 Conn_GPIO, J12 jumper_5v, J13 Conn_power, J14 Conn_01x04_Pin, J2 USB_C_Receptacle_USB2.0, J3 SJ-3523-SMT, J4 USB_A, J5 USB_A, J6 Micro_SD_Card_Det2, J7 Conn_02x04_Odd_Even, J8 Conn_01x02, J9 USB_C_Receptacle_USB2.0, Q1 Q_NPN_BEC, SW1 204-124ST, SW2 SW_Push, SW4 SW_Push, SW6 SW_Push, SW7 SW_SPDT, SW9 SW_SPDT, U1 Ti60F256, U10 MCP4728, U11 LM4811, U12 PCF85063AT/AY, U13 STUSB4500QTR, U14 Si5351A-B-GT, U15 MC2520Z 25MHz, U16 SN74LVC1T45DCK, U17 TPS2116DRLR, U18 TPS562211DRLR, U19 TPS562211DRLR, U2 IM8G16D3FFBG, U20 TPS562211DRLR, U21 TPS562211DRLR, U22 TPS562211DRLR, U23 SN74LVC1T45DCK, U24 SN74LVC1T45DCK, U25 SN74LVC1T45DCK, U3 TFP410PAP, U4 W25Q128JWS, U5 FT2232HL, U6 AP22653W6-7, U7 AP22653W6-7, U8 ESP32-C3-WROOM-02-N4, U9 AP22653W6-7, Y1 12MHz, Y2 Crystal, Y3 25MHz

Commit message: Production files in ../hardware/board_2a
Routing:
- net GND: track 483.6 -> 477.6 mm, vias 207 -> 214
- net Net-(J10-Pin_3): track 20.8 -> 25.1 mm
- net Net-(J10-Pin_1): track 42.5 -> 46.5 mm
- removed copper zone on F.Cu, net (none)
Other:
- board text added: "Endeavour 2a~"
- board text added: "USB1"
- board text added: "USB2"
- board text removed: "Endeavour 2a"
