File: hardware/board_2b/conf.kicad_sch (KiCad schematic)
At the start: 59 parts, among them J7 Conn_02x04_Odd_Even, Q1 Q_NPN_BEC, SW1 204-124ST, SW2 SW_Push, SW3 SW_Push, SW4 SW_Push, SW6 SW_Push, U1 Ti60F256, U14 Si5351A-B-GT, U15 MC2520Z 25MHz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

Commit message: Update hardware/board_2b
Parts:
- D1: value LED -> 5988E20107F
- D2, D3, D4, D5, D6: value LED -> 5988E40107F
- FB1, FB2: value ~ -> 120
- Q1: value Q_NPN_BEC -> Q_NPN_BEC 2SC3326-B,LF
- SW2: value SW_Push -> SW_Push TS02
- SW3, SW4, SW6: value SW_Push -> SW_Push TS11
- Y1: value 12MHz -> ECS120-20-3XTR 12MHz
- Y3: value 25MHz -> ECS250-20-3XTR 25MHz
Changed lines of the file:
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@@
 			)
 		)
-		(property "Value" "SW_Push"
+		(property "Value" "SW_Push TS11"
 			(at 116.205 50.165 0)
 			(effects
@@
 			)
 		)
-		(property "Value" "LED"
-			(at 162.56 167.9574 90)
+		(property "Value" "5988E40107F"
+			(at 167.132 168.148 0)
 			(effects
 				(font
@@
 			)
 		)
-		(property "Value" "LED"
+		(property "Value" "5988E20107F"
 			(at 220.345 84.1374 90)
 			(effects
@@
 			)
 		)
-		(property "Value" "LED"
-			(at 135.255 167.9574 90)
+		(property "Value" "5988E40107F"
+			(at 139.446 168.148 0)
 			(effects
 				(font
@@
 			)
 		)
-		(property "Value" "LED"
+		(property "Value" "5988E40107F"
 			(at 260.35 40.9574 90)
 			(effects
@@
 			)
 		)
-		(property "Value" "~"
-			(at 34.3281 58.42 90)
+		(property "Value" "120"
+			(at 37.592 61.468 90)
 			(effects
 				(font
@@
 			)
 		)
-		(property "Value" "~"
-			(at 34.3281 64.135 90)
+		(property "Value" "120"
+			(at 37.592 66.802 90)
 			(effects
 				(font
@@
 			)
 		)
-		(property "Value" "SW_Push"
+		(property "Value" "SW_Push TS11"
 			(at 116.205 40.005 0)
 			(effects
@@
 			)
 		)
-		(property "Value" "SW_Push"
+		(property "Value" "SW_Push TS02"
 			(at 267.97 79.375 0)
 			(effects
@@
 			)
 		)
-		(property "Value" "25MHz"
+		(property "Value" "ECS250-20-3XTR 25MHz"
 			(at 26.035 30.48 0)
 			(effects
@@
 		(on_board yes)
 		(dnp no)
-		(fields_autoplaced yes)
 		(property "Reference" "Q1"
 			(at 266.065 48.8949 0)
@@
 			)
 		)
-		(property "Value" "Q_NPN_BEC"
-			(at 266.065 51.4349 0)
+		(property "Value" "Q_NPN_BEC 2SC3326-B,LF"
+			(at 270.002 61.214 90)
 			(effects
 				(font
@@
 			)
 		)
-		(property "Value" "12MHz"
+		(property "Value" "ECS120-20-3XTR 12MHz"
 			(at 32.385 162.56 0)
 			(effects
@@
 			)
 		)
-		(property "Value" "SW_Push"
+		(property "Value" "SW_Push TS11"
 			(at 116.205 30.48 0)
 			(effects
@@
 			)
 		)
-		(property "Value" "LED"
-			(at 153.035 167.9574 90)
+		(property "Value" "5988E40107F"
+			(at 157.734 168.402 0)
 			(effects
 				(font
@@
 			)
 		)
-		(property "Value" "LED"
-			(at 144.145 167.9574 90)
+		(property "Value" "5988E40107F"
+			(at 148.336 168.148 0)
 			(effects
 				(font
