File: hardware/board_2b/endeavour2.kicad_sch (KiCad schematic)
At the start: 31 parts, among them J11 Conn_GPIO, J12 Fan, J14 Conn_01x04_Pin, J2 USB_C_Receptacle_USB2.0, J9 Battery, SW9 SW_SPDT, U1 Ti60F256, U12 PCF85063AT/AY, U13 MCP3221/MCP3021, U21 MCP73871-2CC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

Commit message: Update hardware/board_2b
Parts:
- removed D16: LED, LED_SMD:LED_0603_1608Metric, symbol Device:LED
- removed R52: 510, Resistor_SMD:R_0603_1608Metric, symbol Device:R
- D10, D11: value D_TVS -> D_TVS 3v3
- D17: value LED -> 5988E20107F
- D18: value LED -> 5988E40107F
- R51, R70: value 510 -> 560
- SW9: value SW_SPDT -> MSS 3111 D-R
- U12: value PCF85063AT/AY -> PCF85063AT
- Y2: value Crystal -> CM315D32768HZFT
Connections:
- net E2417_SDA is gone; now on net E2417_SCL: U1.B9 (GPIOT_N_09_CLK6_N)
- net E2417_CSB: now also U1.A9 (GPIOT_P_09_CLK6_P); no longer U1.F9 (GPIOT_N_11)
- net E2417_DC: now also U1.C10 (GPIOT_P_12); no longer U1.B10 (GPIOT_P_10_CLK7_P)
- net E2417_RST_N: now also U1.B10 (GPIOT_P_10_CLK7_P); no longer U1.A11 (GPIOT_P_13)
- net E2417_SCL: no longer U1.A9 (GPIOT_P_09_CLK6_P)
- net GPIO_D10: now also J11.10 (Pin_10); no longer J11.9 (Pin_9)
- removed net GPIO_C10: J11.10 (Pin_10), U1.C10 (GPIOT_P_12)
- new net ESP32_DR: U1.A11 (GPIOT_P_13)
- new net GPIO_F9: J11.9 (Pin_9), U1.F9 (GPIOT_N_11)
- no-connect marks 16 -> 17
Changed lines of the file:
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@@
 	)
 	(junction
-		(at 142.875 25.4)
-		(diameter 0)
-		(color 0 0 0 0)
-	)
-	(junction
 		(at 68.58 51.435)
 		(diameter 0)
@@
 	)
 	(no_connect
+		(at 139.065 73.025)
+	)
+	(no_connect
 		(at 54.61 71.755)
 	)
@@
 	(wire
 		(pts
-			(xy 142.875 25.4) (xy 142.875 28.575)
-		)
-		(stroke
-			(width 0)
-			(type default)
-		)
-	)
-	(wire
-		(pts
 			(xy 99.06 65.405) (xy 99.06 57.785)
 		)
@@
 	(wire
 		(pts
-			(xy 149.225 25.4) (xy 142.875 25.4)
+			(xy 83.82 25.4) (xy 149.225 25.4)
 		)
 		(stroke
@@
 	(wire
 		(pts
-			(xy 142.875 73.025) (xy 139.065 73.025)
-		)
-		(stroke
-			(width 0)
-			(type default)
-		)
-	)
-	(wire
-		(pts
 			(xy 189.23 52.705) (xy 189.23 57.785)
 		)
@@
 	(wire
 		(pts
-			(xy 142.875 43.815) (xy 142.875 73.025)
-		)
-		(stroke
-			(width 0)
-			(type default)
-		)
-	)
-	(wire
-		(pts
 			(xy 54.61 57.15) (xy 60.325 57.15)
 		)
@@
 	(wire
 		(pts
-			(xy 142.875 25.4) (xy 83.82 25.4)
-		)
-		(stroke
-			(width 0)
-			(type default)
-		)
-	)
-	(wire
-		(pts
 			(xy 243.205 26.67) (xy 243.205 24.13)
 		)
@@
 	(global_label "E2417_DC"
 		(shape input)
-		(at 168.275 122.555 0)
+		(at 168.275 130.175 0)
 		(fields_autoplaced yes)
 		(effects
@@
 		)
 		(property "Intersheetrefs" "${INTERSHEET_REFS}"
-			(at 175.7632 122.555 0)
+			(at 175.7632 130.175 0)
 			(effects
 				(font
@@
 	(global_label "E2417_RST_N"
 		(shape input)
-		(at 168.275 133.985 0)
+		(at 168.275 122.555 0)
 		(fields_autoplaced yes)
 		(effects
@@
 		)
 		(property "Intersheetrefs" "${INTERSHEET_REFS}"
-			(at 177.6864 133.985 0)
+			(at 177.6864 122.555 0)
 			(effects
 				(font
@@
 	(global_label "E2417_SCL"
 		(shape input)
-		(at 168.275 118.745 0)
+		(at 168.275 120.65 0)
 		(fields_autoplaced yes)
 		(effects
@@
 		)
 		(property "Intersheetrefs" "${INTERSHEET_REFS}"
-			(at 176.3438 118.745 0)
+			(at 176.3438 120.65 0)
 			(effects
 				(font
@@
 		)
 	)
-	(global_label "GPIO_D10"
+	(global_label "GPIO_F9"
 		(shape input)
 		(at 35.56 132.08 180)
@@
 		)
 		(property "Intersheetrefs" "${INTERSHEET_REFS}"
-			(at 25.8666 132.08 0)
+			(at 26.9793 132.08 0)
 			(effects
 				(font
@@
 		)
 	)
-	(global_label "GPIO_C10"
+	(global_label "GPIO_F9"
 		(shape input)
-		(at 168.275 130.175 0)
+		(at 168.275 128.27 0)
 		(fields_autoplaced yes)
 		(effects
@@
 		)
 		(property "Intersheetrefs" "${INTERSHEET_REFS}"
-			(at 175.5456 130.175 0)
+			(at 174.711 128.27 0)
 			(effects
 				(font
@@
 		)
 	)
+	(global_label "ESP32_DR"
+		(shape input)
+		(at 168.275 133.985 0)
+		(fields_autoplaced yes)
+		(effects
+			(font
+				(size 0.762 0.762)
+			)
+			(justify left)
+		)
+		(property "Intersheetrefs" "${INTERSHEET_REFS}"
+			(at 175.7995 133.985 0)
+			(effects
+				(font
+					(size 1.27 1.27)
+				)
+				(justify left)
+				(hide yes)
+			)
+		)
+	)
 	(global_label "GPIO_D11"
 		(shape input)
@@
 	(global_label "E2417_CSB"
 		(shape input)
-		(at 168.275 128.27 0)
+		(at 168.275 118.745 0)
 		(fields_autoplaced yes)
 		(effects
@@
 		)
 		(property "Intersheetrefs" "${INTERSHEET_REFS}"
-			(at 176.4889 128.27 0)
+			(at 176.4889 118.745 0)
 			(effects
 				(font
@@
 		)
 	)
-	(global_label "GPIO_C10"
+	(global_label "GPIO_D10"
 		(shape input)
 		(at 48.26 132.08 0)
@@
 		)
 	)
-	(global_label "E2417_SDA"
-		(shape input)
-		(at 168.275 120.65 0)
-		(fields_autoplaced yes)
-		(effects
-			(font
-				(size 0.762 0.762)
-			)
-			(justify left)
-		)
-		(property "Intersheetrefs" "${INTERSHEET_REFS}"
-			(at 176.38 120.65 0)
-			(effects
-				(font
-					(size 1.27 1.27)
-				)
-				(justify left)
-				(hide yes)
-			)
-		)
-	)
 	(global_label "GPIO_E9"
 		(shape input)
@@
 			)
 		)
-		(property "Value" "510"
+		(property "Value" "560"
 			(at 149.225 41.783 90)
 			(effects
@@
 			)
 		)
-		(property "Value" "510"
+		(property "Value" "560"
 			(at 155.575 41.783 90)
 			(effects
@@
 	)
 	(symbol
-		(lib_id "Device:R")
-		(at 142.875 40.005 0)
-		(unit 1)
-		(exclude_from_sim no)
-		(in_bom yes)
-		(on_board yes)
-		(dnp no)
-		(property "Reference" "R52"
-			(at 140.462 42.164 90)
-			(effects
-				(font
-					(size 1.27 1.27)
-				)
-				(justify left)
-			)
-		)
-		(property "Value" "510"
-			(at 142.875 41.783 90)
-			(effects
-				(font
-					(size 1.27 1.27)
-				)
-				(justify left)
-			)
-		)
-		(property "Footprint" "Resistor_SMD:R_0603_1608Metric"
-			(at 141.097 40.005 90)
-			(effects
-				(font
-					(size 1.27 1.27)
-				)
-				(hide yes)
-			)
-		)
-		(property "Datasheet" "~"
-			(at 142.875 40.005 0)
-			(effects
-				(font
-					(size 1.27 1.27)
-				)
-				(hide yes)
-			)
-		)
-		(property "Description" "Resistor"
-			(at 142.875 40.005 0)
-			(effects
-				(font
-					(size 1.27 1.27)
-				)
-				(hide yes)
-			)
-		)
-		(pin "1"
-		)
-		(pin "2"
-		)
-		(instances
-			(project "endeavour2"
-				(path "/3f72371b-702d-4dab-a6c7-f93a430e8a08"
-					(reference "R52")
-					(unit 1)
-				)
-			)
-		)
-	)
-	(symbol
 		(lib_id "Device:D_TVS")
 		(at 60.325 78.74 90)
@@
 		(on_board yes)
 		(dnp no)
-		(fields_autoplaced yes)
 		(property "Reference" "D10"
 			(at 62.865 77.4699 90)
@@
 			)
 		)
-		(property "Value" "D_TVS"
-			(at 62.865 80.0099 90)
+		(property "Value" "D_TVS 3v3"
+			(at 63.5 78.994 0)
 			(effects
 				(font
@@
 			)
 		)
-		(property "Value" "PCF85063AT/AY"
+		(property "Value" "PCF85063AT"
 			(at 220.98 48.26 0)
 			(effects
@@
 	)
 	(symbol
-		(lib_id "Device:LED")
-		(at 142.875 32.385 270)
-		(mirror x)
-		(unit 1)
-		(exclude_from_sim no)
-		(in_bom yes)
-		(on_board yes)
-		(dnp no)
-		(property "Reference" "D16"
-			(at 142.24 29.845 90)
-			(effects
-				(font
-					(size 1.27 1.27)
-				)
-				(justify right)
-			)
-		)
-		(property "Value" "LED"
-			(at 139.954 31.242 0)
-			(effects
-				(font
-					(size 1.27 1.27)
-				)
-				(justify right)
-			)
-		)
-		(property "Footprint" "LED_SMD:LED_0603_1608Metric"
-			(at 142.875 32.385 0)
-			(effects
-				(font
-					(size 1.27 1.27)
-				)
-				(hide yes)
-			)
-		)
-		(property "Datasheet" "~"
-			(at 142.875 32.385 0)
-			(effects
-				(font
-					(size 1.27 1.27)
-				)
-				(hide yes)
-			)
-		)
-		(property "Description" "Light emitting diode"
-			(at 142.875 32.385 0)
-			(effects
-				(font
-					(size 1.27 1.27)
-				)
-				(hide yes)
-			)
-		)
-		(pin "2"
-		)
-		(pin "1"
-		)
-		(instances
-			(project "endeavour2"
-				(path "/3f72371b-702d-4dab-a6c7-f93a430e8a08"
-					(reference "D16")
-					(unit 1)
-				)
-			)
-		)
-	)
-	(symbol
 		(lib_id "Device:C")
 		(at 251.46 55.245 90)
@@
 			)
 		)
-		(property "Value" "LED"
-			(at 152.654 31.242 0)
+		(property "Value" "5988E40107F"
+			(at 156.718 17.526 0)
 			(effects
 				(font
@@
 			)
 		)
-		(property "Value" "D_TVS"
-			(at 50.165 80.01 90)
+		(property "Value" "D_TVS 3v3"
+			(at 54.356 79.248 0)
 			(effects
 				(font
@@
 			)
 		)
-		(property "Value" "SW_SPDT"
+		(property "Value" "MSS 3111 D-R"
 			(at 170.18 37.465 0)
 			(effects
@@
 			)
 		)
-		(property "Value" "Crystal"
+		(property "Value" "CM315D32768HZFT"
 			(at 193.04 48.26 0)
 			(effects
@@
 			)
 		)
-		(property "Value" "LED"
-			(at 146.304 31.242 0)
+		(property "Value" "5988E20107F"
+			(at 150.368 17.272 0)
 			(effects
 				(font
