File: hardware/board_2b/peripherals.kicad_sch (KiCad schematic)
At the start: 55 parts, among them J3 SJ-3523-SMT, J4 USB_A, J5 USB_A, J6 Micro_SD_Card_Det2, J8 Conn_01x02, SW7 SW_SPDT, U1 Ti60F256, U10 MCP4728, U11 LM4811, U17 TPS2116DRLR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

Commit message: Update hardware/board_2b
Parts:
- added C100, C101: 0.1uF, Capacitor_SMD:C_0603_1608Metric, symbol Device:C
- added U24: SN74LVC2T45DCTR, Package_SO:MSOP-8_3x3mm_P0.65mm, symbol Logic_LevelTranslator:SN74LVC2T45DCUR
- D12, D13, D14, D15: value D_TVS -> D_TVS 3v3
- SW7: value SW_SPDT -> SW_SPDT SLW-864587-2A-RA-N-D
- U31: value SN74LVC2T45DCUR -> SN74LVC2T45DCTR; footprint Package_SO:VSSOP-8_2.3x2mm_P0.5mm -> Package_SO:MSOP-8_3x3mm_P0.65mm
Connections:
- net +1V8: now also C101.1, U24.8 (VCCB)
- net +3V3: now also C100.1, U24.1 (VCCA)
- net ESP32_EN_3V3: now also U24.3 (A2)
- net GND: now also C100.2, C101.2, U24.4 (GND), U24.5 (DIR)
- net ESP32_DR renamed E2417_SDA
- net E2417_SDA: no longer R60.1
- new net CRESET_N: U24.7 (B1)
- new net CRESET_N_3V3: U24.2 (A1)
- new net ESP32_DR_3V3: R60.1
- new net ESP32_EN: U24.6 (B2)
Other:
- moved on the sheet: U1H, U31
