File: hardware/board_2b/ram.kicad_sch (KiCad schematic)
At the start: 36 parts, among them J1 HDMI_A, U1 Ti60F256, U2 IM8G16D3FFBG, U3 TFP410PAP, U9 AP22653W6-7

Commit message: Update hardware/board_2b
Parts:
- removed JP2, JP3: Jumper_2_Bridged, Jumper:SolderJumper-2_P1.3mm_Open_RoundedPad1.0x1.5mm, symbol Jumper:Jumper_2_Open
- added C97: 0.1uF, Capacitor_SMD:C_0603_1608Metric, symbol Device:C
- added R77: 1K, Resistor_SMD:R_0603_1608Metric, symbol Device:R
- added R78: 200K, Resistor_SMD:R_0603_1608Metric, symbol Device:R
- added R79, R80: 2K, Resistor_SMD:R_0603_1608Metric, symbol Device:R
- added U25: PCA9306DP, Package_SO:TSSOP-8_3x3mm_P0.65mm, symbol Interface:PCA9306DP
Connections:
- net +3V3: now also U25.2 (VREF1); no longer U3.13 (ISEL/~{RST})
- net +5V: now also R78.1, R79.1, R80.1
- net 3V3_SCL: now also U25.3 (SCL1)
- net 3V3_SDA: now also U25.4 (SDA1)
- net GND: now also C97.2, U25.1 (GND)
- net at U3.9 (EDGE/HTPLG): now also R77.1
- net at J1.15 (SCL): now also R79.2, U25.6 (SCL2)
- net at J1.16 (SDA): now also R80.2, U25.5 (SDA2)
- net at J1.19 (HPD): now also R77.2
- new net: C97.1, R78.2, U25.7 (VREF2), U25.8 (EN)
- new net CRESET_N_3V3: U3.13 (ISEL/~{RST})
- no-connect marks 20 -> 18
Other:
- moved on the sheet: C32, C33, C34, C35, C36, C40, C42, R45, U9
